Commit message: Upadte config files

File: rm_pioneer_description/urdf/gimbal.urdf.xacro (robot description, xacro)
@@ -5,7 +5,7 @@
   <link name="yaw_link">
     <inertial>
-      <origin xyz="4.9495E-05 -0.036761 0.08872" rpy="0 0 0" />
-      <mass value="0.95681" />
-      <inertia ixx="0.00078388" ixy="-3.16E-06" ixz="1.0358E-07" iyy="0.00060194" iyz="1.0262E-06" izz="0.0010962" />
+      <origin xyz="5.0062E-05 -0.037182 0.086352" rpy="0 0 0" />
+      <mass value="0.94598" />
+      <inertia ixx="0.00078332" ixy="-3.16E-06" ixz="1.0358E-07" iyy="0.00060083" iyz="1.0262E-06" izz="0.0010957" />
     </inertial>
     <visual>
@@ -33,7 +33,7 @@
   <link name="pitch_link">
     <inertial>
-      <origin xyz="0.17934 0.00065681 0.085255" rpy="0 0 0" />
-      <mass value="5.2591" />
-      <inertia ixx="0.022381" ixy="1.1737E-05" ixz="8.3773E-06" iyy="0.016702" iyz="2.0931E-06" izz="0.020886" />
+      <origin xyz="0.034297 0.0026027 0.035447" rpy="0 0 0" />
+      <mass value="1.318" />
+      <inertia ixx="0.0009783" ixy="1.0555E-05" ixz="8.3659E-06" iyy="0.00092518" iyz="2.0079E-06" izz="0.0016519" />
     </inertial>
     <visual>
@@ -54,5 +54,6 @@
   </link>
   <joint name="pitch_joint" type="revolute">
-    <origin xyz="0.0032818 0 0.097945" rpy="0 0 0" />
+    <!-- <origin xyz="0.0032818 0 0.097945" rpy="0 0 0" /> -->
+    <origin xyz="0 0 0.163" rpy="0 0 0" />
     <parent link="yaw_link" />
     <child link="pitch_link" />
@@ -62,5 +63,5 @@
   <link name="shooter_link" />
   <joint name="shooter_joint" type="fixed">
-    <origin xyz="0.0032818 0 0.097945" rpy="0 0 0" />
+    <origin xyz="0 0 0.163" rpy="0 0 0" />
     <parent link="base_link" />
     <child link="shooter_link" />
@@ -68,7 +69,7 @@
   <link name="camera_base_link">
     <inertial>
-      <origin xyz="-0.015408 1.3878E-17 -2.7756E-17" rpy="0 0 0" />
-      <mass value="0.082876" />
-      <inertia ixx="1.7456E-05" ixy="1.0384E-21" ixz="-4.9613E-21" iyy="4.0132E-05" iyz="4.8698E-22" izz="4.0162E-05" />
+      <origin xyz="-0.45111 0.035515 0.068286" rpy="0 0 0" />
+      <mass value="0" />
+      <inertia ixx="0" ixy="0" ixz="0" iyy="0" iyz="0" izz="0" />
     </inertial>
     <visual>
@@ -89,5 +90,5 @@
   </link>
   <joint name="camera_base_joint" type="fixed">
-    <origin xyz="0.088 0.0 0.0585" rpy="0 0 0" />
+    <origin xyz="0.0806 0 0.0518" rpy="0 0 0" />
     <parent link="pitch_link" />
     <child link="camera_base_link" />
